File: Schematics/SAME70CPad.sch (KiCad schematic (older format))
At the start: 204 parts, among them J1 ER-TFTMO70-5-LCD, J10 Headset, J11 MIC_IN, J12 POWER, J13 RESET, J14 BATTERY, J15 PWR_QON, J2 nFL24l02_Module, J3 SWD/JTAG, J4 USB_OTG, J5 DEBUG_UART, J6 ERASE, J7 POWER_IN, J8 SPKRL, J9 SPKRR, M1 MountingHole, M2 MountingHole, M3 MountingHole, M4 MountingHole, P1 ESP-12E, P2 ER-TFTMO70-5-SD, P3 MicroSD, Q1 RE1C002UN, Q2 RE1C002UN, Q3 RE1C002UN, SW1 SW_POWER, U1 IS42S16320D, U10 XC9142B50DMR-G, U11 TPS62063, U12 AP2138N18, U13 bq24297, U14 INA3221AIRGVx, U2 MCP1501T-25E/CHY, U3 IS25LP256D, U4 ATSAME70QxxA-AN, U5 D5V0F4U6SO, U6 TLV320AIC3111, U7 BME280, U8 MPU-9250, U9 ICS-40181, Y1 32.768kHz, Y2 12MHz

Commit message: Added some missing pullup resistors plus misc cleanup and optimization of the layout.
Parts:
- added R46: 100k, MyResistors:R_0603, symbol R_Small
- renumbered C37 to C1, C25 to C10, C24 to C11, C1 to C12, C27 to C13, C38 to C14, C34 to C15, C12 to C16, C2 to C17, C30 to C18, C11 to C19, C14 to C2, C36 to C20, C78 to C21, C74 to C22, C59 to C23, C73 to C24, C60 to C25, C70 to C26, C69 to C27, C21 to C28, C28 to C29, C31 to C3, C84 to C30, C19 to C31, C16 to C32, C29 to C33, C89 to C34, C90 to C35, C91 to C36, C18 to C37, C79 to C38, C17 to C39, C53 to C4, C43 to C40, C66 to C41, C83 to C42, C20 to C43, C3 to C44, C23 to C45, C93 to C46, C13 to C47, C80 to C48, C77 to C49, C35 to C5, C71 to C50, C15 to C51, C26 to C52, C94 to C53, C32 to C54, C52 to C55, C55 to C56, C62 to C57, C65 to C58, C57 to C59, C22 to C6, C39 to C60, C56 to C61, C63 to C62, C40 to C63, C45 to C64, C47 to C65, C50 to C66, C48 to C67, C46 to C68, C49 to C69, C72 to C7, C51 to C70, C44 to C71, C42 to C72, C41 to C73, C82 to C74, C64 to C75, C67 to C76, C68 to C77, C61 to C78, C75 to C79, C33 to C8, C76 to C80, C54 to C81, C81 to C82, C5 to C83, C4 to C84, C87 to C85, C88 to C86, C85 to C87, C86 to C88, C10 to C89, C58 to C9, C6 to C90, C7 to C91, C8 to C92, C9 to C93, C92 to C94, J12 to J1, J2 to J10, J10 to J11, J14 to J12, J11 to J13, J8 to J14, J9 to J15, J13 to J2, J15 to J3, J5 to J4, J3 to J5, J7 to J6, J1 to J7, J4 to J8, J6 to J9, L5 to L1, L1 to L2, L2 to L4, L6 to L5, L4 to L6, M4 to M1, M3 to M2, M1 to M3, M2 to M4, P3 to P1, P1 to P3, R22 to R1, R17 to R10, R20 to R11, R5 to R12, R21 to R13, R36 to R14, R35 to R15, R4 to R16, R39 to R17, R40 to R18, R41 to R19, R45 to R2, R31 to R20, R33 to R21, R38 to R22, R34 to R23, R27 to R25, R2 to R26, R13 to R27, R9 to R28, R37 to R29, R25 to R3, R32 to R30, R1 to R31, R8 to R32, R12 to R33, R14 to R34, R15 to R35, R11 to R36, R10 to R37, R30 to R38, R6 to R39, R28 to R4, R42 to R40, R43 to R41, R3 to R42, R26 to R43, R18 to R44, R7 to R45, R29 to R5, R23 to R6, R44 to R7, R19 to R8, R16 to R9, RN13 to RN1, RN7 to RN10, RN4 to RN11, RN1 to RN12, RN5 to RN13, RN2 to RN14, RN9 to RN2, RN14 to RN3, RN12 to RN4, RN3 to RN5, RN11 to RN7, RN10 to RN9, U3 to U1, U9 to U10, U6 to U11, U10 to U12, U12 to U13, U1 to U14, U8 to U3, U13 to U4, U4 to U5, U5 to U6, U14 to U7, U11 to U8, U7 to U9
Connections:
- net +3V3: now also R46.2
- net QSPI_CE: now also R46.1

Commit message: - Annotated components geographically from the PCB layout. - Added the OSHW logo to the PCB. - Some minor layout cleanup.
Parts:
- renumbered C22 to C15, C21 to C16, C23 to C17, C15 to C18, C16 to C19, C3 to C2, C17 to C20, C18 to C21, C19 to C22, C20 to C23, C2 to C3, C32 to C31, C31 to C32, C35 to C34, C34 to C35, C40 to C39, C7 to C4, C39 to C40, C48 to C46, C49 to C47, C46 to C48, C47 to C49, C4 to C5, C58 to C57, C59 to C58, C60 to C59, C57 to C60, C63 to C62, C62 to C63, C71 to C69, C5 to C7, C69 to C70, C70 to C71, C74 to C72, C78 to C73, C75 to C74, C72 to C75, C73 to C76, C76 to C77, C77 to C78, C9 to C8, C82 to C81, C81 to C82, C8 to C9, J11 to J10, J10 to J11, R3 to R2, R46 to R21, R21 to R22, R22 to R23, R23 to R24, R24 to R25, R25 to R26, R26 to R28, R28 to R29, R4 to R3, R29 to R30, R30 to R31, R31 to R32, R32 to R33, R33 to R34, R34 to R35, R35 to R36, R36 to R37, R37 to R38, R38 to R39, R5 to R4, R39 to R40, R40 to R41, R41 to R42, R42 to R43, R43 to R44, R44 to R45, R45 to R46, R6 to R5, R2 to R6
